File: Hardware/PCB/front.kicad_sch (KiCad schematic)
At the start: 28 parts, among them SW901 SW_SPDT_MSM, U1 TL072, U2 TL072

Commit message: Layout redone
Parts:
- added H903, H904: MountingHole, ao_tht:MountingHole_3.2mm_M3, symbol ao_symbols:MountingHole
- added TP904: +12V, ao_tht:TestPoint_THTPad_D1.5mm_Drill0.7mm, symbol ao_symbols:TestPoint
- added TP905: GND, ao_tht:TestPoint_THTPad_D1.5mm_Drill0.7mm, symbol ao_symbols:TestPoint
- added TP906: -12V, ao_tht:TestPoint_THTPad_D1.5mm_Drill0.7mm, symbol ao_symbols:TestPoint
Connections:
- net +12V: now also TP904.1
- net -12V: now also TP906.1
- net GND: now also TP905.1
Changed lines of the file:
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@@
+    (pin "1")
+  )
+  (symbol (lib_id "power:-12V") (at 96.52 172.72 180) (unit 1)
+    (in_bom yes) (on_board yes) (fields_autoplaced)
+    (property "Reference" "#PWR0149" (id 0) (at 96.52 175.26 0)
+      (effects (font (size 1.27 1.27)) hide)
+    )
+    (property "Value" "-12V" (id 1) (at 96.52 177.1634 0))
+    (property "Footprint" "" (id 2) (at 96.52 172.72 0)
+      (effects (font (size 1.27 1.27)) hide)
+    )
+    (property "Datasheet" "" (id 3) (at 96.52 172.72 0)
+      (effects (font (size 1.27 1.27)) hide)
+    )
     (pin "1")
   )
@@
     (pin "1")
   )
+  (symbol (lib_id "power:GND") (at 82.55 172.72 0) (unit 1)
+    (in_bom yes) (on_board yes)
+    (property "Reference" "#SUPPLY0102" (id 0) (at 82.55 172.72 0)
+      (effects (font (size 1.27 1.27)) hide)
+    )
+    (property "Value" "GND" (id 1) (at 82.55 176.53 0))
+    (property "Footprint" "" (id 2) (at 82.55 172.72 0)
+      (effects (font (size 1.27 1.27)) hide)
+    )
+    (property "Datasheet" "" (id 3) (at 82.55 172.72 0)
+      (effects (font (size 1.27 1.27)) hide)
+    )
+    (pin "1")
+  )
   (symbol (lib_id "power:GND") (at 45.72 40.64 0) (unit 1)
     (in_bom yes) (on_board yes)
@@
     (pin "2")
     (pin "3")
+  )
+  (symbol (lib_id "ao_symbols:TestPoint") (at 82.55 172.72 0) (unit 1)
+    (in_bom no) (on_board yes) (fields_autoplaced)
+    (property "Reference" "TP905" (id 0) (at 83.947 168.5833 0)
+      (effects (font (size 1.27 1.27)) (justify left))
+    )
+    (property "Value" "GND" (id 1) (at 83.947 171.1202 0)
+      (effects (font (size 1.27 1.27)) (justify left))
+    )
+    (property "Footprint" "ao_tht:TestPoint_THTPad_D1.5mm_Drill0.7mm" (id 2) (at 87.63 172.72 0)
+      (effects (font (size 1.27 1.27)) hide)
+    )
+    (property "Datasheet" "~" (id 3) (at 87.63 172.72 0)
+      (effects (font (size 1.27 1.27)) hide)
+    )
+    (property "Config" "DNF" (id 4) (at 82.55 172.72 0)
+      (effects (font (size 1.27 1.27)) hide)
+    )
+    (pin "1")
   )
   (symbol (lib_id "ao_symbols:TL072") (at 243.84 156.21 0) (unit 3)
@@
     (pin "3")
   )
+  (symbol (lib_id "ao_symbols:TestPoint") (at 96.52 172.72 0) (unit 1)
+    (in_bom no) (on_board yes) (fields_autoplaced)
+    (property "Reference" "TP906" (id 0) (at 97.917 168.5833 0)
+      (effects (font (size 1.27 1.27)) (justify left))
+    )
+    (property "Value" "-12V" (id 1) (at 97.917 171.1202 0)
+      (effects (font (size 1.27 1.27)) (justify left))
+    )
+    (property "Footprint" "ao_tht:TestPoint_THTPad_D1.5mm_Drill0.7mm" (id 2) (at 101.6 172.72 0)
+      (effects (font (size 1.27 1.27)) hide)
+    )
+    (property "Datasheet" "~" (id 3) (at 101.6 172.72 0)
+      (effects (font (size 1.27 1.27)) hide)
+    )
+    (property "Config" "DNF" (id 4) (at 96.52 172.72 0)
+      (effects (font (size 1.27 1.27)) hide)
+    )
+    (pin "1")
+  )
   (symbol (lib_id "power:+12V") (at 147.32 81.28 0) (unit 1)
     (in_bom yes) (on_board yes)
@@
     )
     (property "Datasheet" "" (id 3) (at 147.32 81.28 0)
+      (effects (font (size 1.27 1.27)) hide)
+    )
+    (pin "1")
+  )
+  (symbol (lib_id "power:+12V") (at 71.12 171.45 0) (unit 1)
+    (in_bom yes) (on_board yes)
+    (property "Reference" "#PWR0150" (id 0) (at 71.12 175.26 0)
+      (effects (font (size 1.27 1.27)) hide)
+    )
+    (property "Value" "+12V" (id 1) (at 71.12 167.8742 0))
+    (property "Footprint" "" (id 2) (at 71.12 171.45 0)
+      (effects (font (size 1.27 1.27)) hide)
+    )
+    (property "Datasheet" "" (id 3) (at 71.12 171.45 0)
       (effects (font (size 1.27 1.27)) hide)
     )
@@
     (pin "1")
   )
+  (symbol (lib_id "ao_symbols:TestPoint") (at 71.12 171.45 0) (mirror x) (unit 1)
+    (in_bom no) (on_board yes) (fields_autoplaced)
+    (property "Reference" "TP904" (id 0) (at 69.723 173.9173 0)
+      (effects (font (size 1.27 1.27)) (justify right))
+    )
+    (property "Value" "+12V" (id 1) (at 69.723 176.4542 0)
+      (effects (font (size 1.27 1.27)) (justify right))
+    )
+    (property "Footprint" "ao_tht:TestPoint_THTPad_D1.5mm_Drill0.7mm" (id 2) (at 76.2 171.45 0)
+      (effects (font (size 1.27 1.27)) hide)
+    )
+    (property "Datasheet" "~" (id 3) (at 76.2 171.45 0)
+      (effects (font (size 1.27 1.27)) hide)
+    )
+    (property "Config" "DNF" (id 4) (at 71.12 171.45 0)
+      (effects (font (size 1.27 1.27)) hide)
+    )
+    (pin "1")
+  )
   (symbol (lib_id "power:GND") (at 221.615 156.21 0) (unit 1)
     (in_bom yes) (on_board yes) (fields_autoplaced)
@@
     (pin "1")
   )
+  (symbol (lib_id "ao_symbols:MountingHole") (at 132.08 168.91 0) (unit 1)
+    (in_bom no) (on_board yes) (fields_autoplaced)
+    (property "Reference" "H904" (id 0) (at 134.62 168.0753 0)
+      (effects (font (size 1.27 1.27)) (justify left))
+    )
+    (property "Value" "MountingHole" (id 1) (at 134.62 170.6122 0)
+      (effects (font (size 1.27 1.27)) (justify left))
+    )
+    (property "Footprint" "ao_tht:MountingHole_3.2mm_M3" (id 2) (at 132.08 168.91 0)
+      (effects (font (size 1.27 1.27)) hide)
+    )
+    (property "Datasheet" "" (id 3) (at 132.08 168.91 0)
+      (effects (font (size 1.27 1.27)) hide)
+    )
+    (property "Config" "DNF" (id 4) (at 132.08 168.91 0)
+      (effects (font (size 1.27 1.27)) hide)
+    )
+  )
+  (symbol (lib_id "ao_symbols:MountingHole") (at 113.03 168.91 0) (unit 1)
+    (in_bom no) (on_board yes) (fields_autoplaced)
+    (property "Reference" "H903" (id 0) (at 115.57 168.0753 0)
+      (effects (font (size 1.27 1.27)) (justify left))
+    )
+    (property "Value" "MountingHole" (id 1) (at 115.57 170.6122 0)
+      (effects (font (size 1.27 1.27)) (justify left))
+    )
+    (property "Footprint" "ao_tht:MountingHole_3.2mm_M3" (id 2) (at 113.03 168.91 0)
+      (effects (font (size 1.27 1.27)) hide)
+    )
+    (property "Datasheet" "" (id 3) (at 113.03 168.91 0)
+      (effects (font (size 1.27 1.27)) hide)
+    )
+    (property "Config" "DNF" (id 4) (at 113.03 168.91 0)
+      (effects (font (size 1.27 1.27)) hide)
+    )
+  )
   (symbol (lib_id "ao_symbols:R") (at 129.54 76.2 0) (unit 1)
