File: Hardware/SpringReverbRev2/PCB/springReverbRev2.kicad_sch (KiCad schematic)
At the start: 12 parts, among them J1 Conn_01x08, J2 Conn_01x08

Commit message: misc corrections
Parts:
- J1: footprint Connector_PinSocket_2.54mm:PinSocket_1x09_P2.54mm_Vertical -> Connector_PinSocket_2.54mm:PinSocket_1x08_P2.54mm_Vertical
Changed lines of the file:
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@@
     (property "Reference" "J1" (id 0) (at 129.54 66.1502 0))
     (property "Value" "Conn_01x08" (id 1) (at 129.54 68.6871 0))
-    (property "Footprint" "Connector_PinSocket_2.54mm:PinSocket_1x09_P2.54mm_Vertical" (id 2) (at 129.54 81.28 0)
+    (property "Footprint" "Connector_PinSocket_2.54mm:PinSocket_1x08_P2.54mm_Vertical" (id 2) (at 129.54 81.28 0)
       (effects (font (size 1.27 1.27)) hide)
     )
@@
     )
     (path "/cb7e7ca4-1a75-4992-9aba-d7df48630a9d/2a64b8ca-30ae-497f-8920-bdcfda6b245c"
-      (reference "C1") (unit 1) (value "10uf") (footprint "ao_tht:CP_Radial_D6.3mm_P2.50mm")
+      (reference "C1") (unit 1) (value "10uF") (footprint "ao_tht:C_Disc_D3.0mm_W1.6mm_P2.50mm")
     )
     (path "/cb7e7ca4-1a75-4992-9aba-d7df48630a9d/292c0221-0e8e-434d-bc93-686854d7557e"
-      (reference "C2") (unit 1) (value "10uf") (footprint "ao_tht:CP_Radial_D6.3mm_P2.50mm")
+      (reference "C2") (unit 1) (value "10uF") (footprint "ao_tht:C_Disc_D3.0mm_W1.6mm_P2.50mm")
     )
     (path "/cb7e7ca4-1a75-4992-9aba-d7df48630a9d/58a249a3-3637-43bb-891c-d8fb3aea2eb1"
@@
     )
     (path "/757cdb0d-1f9d-4951-b906-b680c7b834f3/a4ef3478-d779-4ed7-919b-261c438a0472"
-      (reference "C6") (unit 1) (value "100n") (footprint "ao_tht:C_Disc_D3.0mm_W1.6mm_P2.50mm")
+      (reference "C6") (unit 1) (value "100nF") (footprint "ao_tht:C_Disc_D3.0mm_W1.6mm_P2.50mm")
     )
     (path "/757cdb0d-1f9d-4951-b906-b680c7b834f3/6f296ea0-4d2f-46eb-b08c-bf8505fb155a"
-      (reference "C7") (unit 1) (value "100n") (footprint "ao_tht:C_Disc_D3.0mm_W1.6mm_P2.50mm")
+      (reference "C7") (unit 1) (value "100nF") (footprint "ao_tht:C_Disc_D3.0mm_W1.6mm_P2.50mm")
     )
     (path "/cb7e7ca4-1a75-4992-9aba-d7df48630a9d/b44557fd-b109-46e6-9c47-7898fc72d72b"
-      (reference "C101") (unit 1) (value "10uF") (footprint "ao_tht:CP_Radial_D6.3mm_P2.50mm")
+      (reference "C101") (unit 1) (value "10uF") (footprint "ao_tht:C_Disc_D3.0mm_W1.6mm_P2.50mm")
     )
     (path "/a1f902c6-fb29-4830-82ac-958ceff67f3f"
@@
     )
     (path "/cb7e7ca4-1a75-4992-9aba-d7df48630a9d/abdccd32-4761-4905-9e3c-5822fd231b2c"
-      (reference "C104") (unit 1) (value "100n") (footprint "ao_tht:C_Disc_D3.0mm_W1.6mm_P2.50mm")
+      (reference "C104") (unit 1) (value "100nF") (footprint "ao_tht:C_Disc_D3.0mm_W1.6mm_P2.50mm")
     )
     (path "/cb7e7ca4-1a75-4992-9aba-d7df48630a9d/ba9f5381-b220-49fe-a059-7479eebb8012"
-      (reference "C105") (unit 1) (value "100n") (footprint "ao_tht:C_Disc_D3.0mm_W1.6mm_P2.50mm")
+      (reference "C105") (unit 1) (value "100nF") (footprint "ao_tht:C_Disc_D3.0mm_W1.6mm_P2.50mm")
     )
     (path "/cb7e7ca4-1a75-4992-9aba-d7df48630a9d/8aef1f5e-d708-477f-85a2-d00886ea3b16"
-      (reference "C106") (unit 1) (value "100n") (footprint "ao_tht:C_Disc_D3.0mm_W1.6mm_P2.50mm")
+      (reference "C106") (unit 1) (value "100nF") (footprint "ao_tht:C_Disc_D3.0mm_W1.6mm_P2.50mm")
     )
     (path "/cb7e7ca4-1a75-4992-9aba-d7df48630a9d/09d29258-41fc-4a62-9201-ea401458f7b0"
-      (reference "C107") (unit 1) (value "100n") (footprint "ao_tht:C_Disc_D3.0mm_W1.6mm_P2.50mm")
+      (reference "C107") (unit 1) (value "100nF") (footprint "ao_tht:C_Disc_D3.0mm_W1.6mm_P2.50mm")
     )
     (path "/cb7e7ca4-1a75-4992-9aba-d7df48630a9d/80481072-eb6a-4497-9b33-a8933ec1c2b4"
@@
     )
     (path "/cb7e7ca4-1a75-4992-9aba-d7df48630a9d/dfad2ca5-0341-46cc-af98-e92db90ec536"
-      (reference "C109") (unit 1) (value "22uF") (footprint "ao_tht:CP_Radial_D6.3mm_P2.50mm")
+      (reference "C109") (unit 1) (value "22uF") (footprint "ao_tht:C_Disc_D3.0mm_W1.6mm_P2.50mm")
     )
     (path "/cb7e7ca4-1a75-4992-9aba-d7df48630a9d/2affb285-bf40-45c0-bbb0-c2ccfaf4c77b"
@@
     )
     (path "/cb7e7ca4-1a75-4992-9aba-d7df48630a9d/6f26d5ca-6fc6-459b-9376-4778608b6b29"
-      (reference "C901") (unit 1) (value "100n") (footprint "ao_tht:C_Disc_D3.0mm_W1.6mm_P2.50mm")
+      (reference "C901") (unit 1) (value "100nF") (footprint "ao_tht:C_Disc_D3.0mm_W1.6mm_P2.50mm")
     )
     (path "/cb7e7ca4-1a75-4992-9aba-d7df48630a9d/efaea355-f240-4fe6-abb2-f17dca6f3718"
-      (reference "C902") (unit 1) (value "100n") (footprint "ao_tht:C_Disc_D3.0mm_W1.6mm_P2.50mm")
+      (reference "C902") (unit 1) (value "100nF") (footprint "ao_tht:C_Disc_D3.0mm_W1.6mm_P2.50mm")
     )
     (path "/757cdb0d-1f9d-4951-b906-b680c7b834f3/5aa60a7b-85fa-4016-848e-ae69c3ab164a"
-      (reference "C903") (unit 1) (value "100n") (footprint "ao_tht:C_Disc_D3.0mm_W1.6mm_P2.50mm")
+      (reference "C903") (unit 1) (value "100nF") (footprint "ao_tht:C_Disc_D3.0mm_W1.6mm_P2.50mm")
     )
     (path "/757cdb0d-1f9d-4951-b906-b680c7b834f3/6f3c805a-4ac4-4a79-b4d0-0b7ae752167a"
-      (reference "C904") (unit 1) (value "100n") (footprint "ao_tht:C_Disc_D3.0mm_W1.6mm_P2.50mm")
+      (reference "C904") (unit 1) (value "100nF") (footprint "ao_tht:C_Disc_D3.0mm_W1.6mm_P2.50mm")
     )
     (path "/b957cd77-9ec1-4fe1-8d3b-0eb575c216ba"
@@
     )
     (path "/a3231254-9a06-4749-9f8c-d0e0a9e2b786"
-      (reference "J1") (unit 1) (value "Conn_01x08") (footprint "Connector_PinSocket_2.54mm:PinSocket_1x09_P2.54mm_Vertical")
+      (reference "J1") (unit 1) (value "Conn_01x08") (footprint "Connector_PinSocket_2.54mm:PinSocket_1x08_P2.54mm_Vertical")
     )
     (path "/b2cf5a83-4806-4849-a00d-e9939041bf9b"

Commit message: Backlog
Parts:
- removed J1: Conn_01x08, Connector_PinSocket_2.54mm:PinSocket_1x08_P2.54mm_Vertical, symbol Connector_Generic:Conn_01x08
- removed J2: Conn_01x08, Connector_PinHeader_2.54mm:PinHeader_1x08_P2.54mm_Vertical, symbol Connector_Generic:Conn_01x08
- removed JP104: Conn_01x06, Connector_PinHeader_2.54mm:PinHeader_1x06_P2.54mm_Vertical, symbol Connector_Generic:Conn_01x06
- removed JP2: Conn_01x06, Connector_PinSocket_2.54mm:PinSocket_1x06_P2.54mm_Vertical, symbol Connector_Generic:Conn_01x06
- added J907: Conn_01x08_Socket, Connector_PinSocket_2.54mm:PinSocket_1x08_P2.54mm_Vertical, symbol Connector:Conn_01x08_Socket
- added J908: Conn_01x08_Pin, Connector_PinHeader_2.54mm:PinHeader_1x08_P2.54mm_Vertical, symbol Connector:Conn_01x08_Pin
- added J909: Conn_01x09_Socket, Connector_PinSocket_2.54mm:PinSocket_1x09_P2.54mm_Vertical, symbol Connector:Conn_01x09_Socket
- added J910: Conn_01x09_Pin, Connector_PinHeader_2.54mm:PinHeader_1x09_P2.54mm_Vertical, symbol Connector:Conn_01x09_Pin
- added J911, J912: 2_pin_Molex_header, AO_tht:Molex_KK-254_AE-6410-02A_1x02_P2.54mm_Vertical, symbol AO_symbols:2_pin_Molex_header
- added J913, J914: 2_pin_Molex_connector, AO_tht:Molex_KK-254_AE-6410-02A_1x02_P2.54mm_Vertical, symbol AO_symbols:2_pin_Molex_connector
- C102, C103: footprint ao_tht:CP_Radial_D6.3mm_P2.50mm -> AO_tht:CP_Radial_D6.3mm_P2.50mm; symbol ao_symbols:CP -> AO_symbols:CP
- D901, D902: footprint ao_tht:D_DO-41_SOD81_P10.16mm_Horizontal -> AO_tht:D_DO-41_SOD81_P10.16mm_Horizontal; symbol ao_symbols:1N5817 -> AO_symbols:1N5817
- SV101: footprint ao_tht:Power_Header -> AO_tht:Power_Header; symbol ao_symbols:Synth_power_2x5 -> AO_symbols:Synth_power_2x5
- TP901, TP902, TP903: footprint ao_tht:TestPoint_THTPad_D1.5mm_Drill0.7mm -> AO_tht:TestPoint_THTPad_D1.5mm_Drill0.7mm; symbol ao_symbols:TestPoint -> AO_symbols:TestPoint
Connections:
- net +12V: now also J909.2 (Pin_2)
- net +12V_B: now also J910.2 (Pin_2)
- net -12V: now also J909.3 (Pin_3)
- net -12V_B: now also J910.3 (Pin_3)
- net Back board/AUDIO_IN_1: now also J908.5 (Pin_5)
- net Back board/AUDIO_IN_2: now also J908.6 (Pin_6)
- net Back board/CV_IN: now also J908.4 (Pin_4)
- net Back board/DRY_B: now also J908.7 (Pin_7)
- net Back board/EQ_POT_1_B: now also J908.1 (Pin_1)
- net Back board/EQ_POT_2_B: now also J908.2 (Pin_2)
- net Back board/EQ_POT_3_B: now also J908.3 (Pin_3)
- net Back board/TRIM_B: now also J910.4 (Pin_4)
- net Back board/VAC_AN_B: now also J910.5 (Pin_5)
- net Back board/VAC_CA_B: now also J910.6 (Pin_6)
- net Front board/AUDIO_IN_1: now also J907.5 (Pin_5)
- net Front board/AUDIO_IN_2: now also J907.6 (Pin_6)
- net Front board/CV_IN: now also J907.4 (Pin_4)
- net Front board/DRY_F: now also J907.7 (Pin_7)
- net Front board/EQ_POT_1_F: now also J907.1 (Pin_1)
- net Front board/EQ_POT_2_F: now also J907.2 (Pin_2)
- net Front board/EQ_POT_3_F: now also J907.3 (Pin_3)
- net Front board/TRIM_F: now also J909.4 (Pin_4)
- net Front board/VAC_AN_F: now also J909.5 (Pin_5)
- net Front board/VAC_CA_F: now also J909.6 (Pin_6)
- net GND: now also J909.1 (Pin_1)
- net GND_B: now also J910.1 (Pin_1), J912.2 (Pin_2)
- new net Back board/FROM_TANK_T_B: J912.1 (Pin_1)
- new net Back board/MIXPOT_DRY_B: J910.7 (Pin_7)
- new net Back board/MIXPOT_MIX_B: J910.8 (Pin_8)
- new net Back board/MIXPOT_WET_B: J910.9 (Pin_9)
- new net Back board/TO_TANK_S_B: J911.1 (Pin_1)
- new net Back board/TO_TANK_T_B: J911.2 (Pin_2)
- new net Front board/MIXPOT_DRY_F: J909.7 (Pin_7)
- new net Front board/MIXPOT_MIX_F: J909.8 (Pin_8)
- new net Front board/MIXPOT_WET_F: J909.9 (Pin_9)
- new net GND_P: J914.2 (Pin_2)
- new net Panel mount/FROM_TANK_T_P: J914.1 (Pin_1)
- new net Panel mount/TO_TANK_S_P: J913.1 (Pin_1)
- new net Panel mount/TO_TANK_T_P: J913.2 (Pin_2)
Other:
- added sheet Panel mount (panelmount.kicad_sch)
- sheet Back board ports: added FROM_TANK_T_B, MIXPOT_DRY_B, MIXPOT_MIX_B, MIXPOT_WET_B, TO_TANK_S_B, TO_TANK_T_B; removed none
- sheet Front board ports: added MIXPOT_DRY_F, MIXPOT_MIX_F, MIXPOT_WET_F; removed none
