File: Hardware/SpringReverbRev2/PCB/springReverbRev2.kicad_pcb (KiCad board)
At the start: 2 copper layers, 165 x 159.5 mm, 99 parts, among them IC102 TL074, IC103 TL074, J1 Conn_01x08, J2 Conn_01x08, J901 AudioJack2_SwitchT, J902 AudioJack2, J903 AudioJack2, J904 AudioJack2, J905 AudioJack2_SwitchT, J906 AudioJack2, SW901 SW_SPDT_MSM, U1 TL072, U2 TL072, U7 NE5532, U901 L78L05_TO92, X101 RCA, X102 RCA

Commit message: misc corrections
Parts:
- J1: footprint Connector_PinSocket_2.54mm:PinSocket_1x09_P2.54mm_Vertical -> Connector_PinSocket_2.54mm:PinSocket_1x08_P2.54mm_Vertical

Commit message: Backlog
Parts:
- removed H904: MountingHole, ao_tht:MountingHole_3.2mm_M3
- removed J1: Conn_01x08, Connector_PinSocket_2.54mm:PinSocket_1x08_P2.54mm_Vertical
- removed J2: Conn_01x08, Connector_PinHeader_2.54mm:PinHeader_1x08_P2.54mm_Vertical
- removed JP101: Conn_01x04, Connector_Molex:Molex_KK-254_AE-6410-04A_1x04_P2.54mm_Vertical
- removed JP102: Conn_01x03, ao_tht:Molex_KK-254_AE-6410-03A_1x03_P2.54mm_Vertical
- removed JP104: Conn_01x06, Connector_PinHeader_2.54mm:PinHeader_1x06_P2.54mm_Vertical
- removed JP2: Conn_01x06, Connector_PinSocket_2.54mm:PinSocket_1x06_P2.54mm_Vertical
- added H905: MountingHole, AO_tht:MountingHole_3.2mm_M3, F.Cu at (145.0, 31.5)
- added J907: Conn_01x08_Socket, Connector_PinSocket_2.54mm:PinSocket_1x08_P2.54mm_Vertical, B.Cu at (117.8, 67.0)
- added J908: Conn_01x08_Pin, Connector_PinHeader_2.54mm:PinHeader_1x08_P2.54mm_Vertical, F.Cu at (242.8, 67.0)
- added J909: Conn_01x09_Socket, Connector_PinSocket_2.54mm:PinSocket_1x09_P2.54mm_Vertical, B.Cu at (138.1, 108.9)
- added J910: Conn_01x09_Pin, Connector_PinHeader_2.54mm:PinHeader_1x09_P2.54mm_Vertical, F.Cu at (263.1, 108.9)
- added J911: 2_pin_Molex_header, AO_tht:Molex_KK-254_AE-6410-02A_1x02_P2.54mm_Vertical, B.Cu at (243.5, 136.8)
- added J912: 2_pin_Molex_header, AO_tht:Molex_KK-254_AE-6410-02A_1x02_P2.54mm_Vertical, B.Cu at (261.3, 136.8)
- added RV905: B50k, AO_tht:Potentiometer_Alpha_16mm_Single_Vertical, F.Cu at (125.0, 85.0)
- C1, C2: value 10uf -> 10uF; footprint ao_tht:CP_Radial_D6.3mm_P2.50mm -> AO_tht:C_Disc_D3.0mm_W1.6mm_P2.50mm; moved to B.Cu
- C101, C109: footprint ao_tht:CP_Radial_D6.3mm_P2.50mm -> AO_tht:C_Disc_D3.0mm_W1.6mm_P2.50mm; moved to B.Cu
- C102, C103: footprint ao_tht:CP_Radial_D6.3mm_P2.50mm -> AO_tht:CP_Radial_D6.3mm_P2.50mm; moved to B.Cu
- C104, C105, C106, C107, C6, C7, C901, C902, C903, C904: value 100n -> 100nF; footprint ao_tht:C_Disc_D3.0mm_W1.6mm_P2.50mm -> AO_tht:C_Disc_D3.0mm_W1.6mm_P2.50mm; moved to B.Cu
- C108, C110, C3, C4: footprint ao_tht:C_Rect_L7.2mm_W2.5mm_P5.00mm_FKS2_FKP2_MKS2_MKP2 -> AO_tht:C_Disc_D3.0mm_W1.6mm_P2.50mm; moved to B.Cu
- C5: footprint ao_tht:C_Disc_D5.0mm_W2.5mm_P5.00mm -> AO_tht:C_Disc_D3.0mm_W1.6mm_P2.50mm; moved to B.Cu
- D901, D902: footprint ao_tht:D_DO-41_SOD81_P10.16mm_Horizontal -> AO_tht:D_DO-41_SOD81_P10.16mm_Horizontal; moved to B.Cu
- H901, H902, H903: footprint ao_tht:MountingHole_3.2mm_M3 -> AO_tht:MountingHole_3.2mm_M3
- IC102, IC103: footprint ao_tht:DIP-14_W7.62mm_Socket_LongPads -> AO_tht:DIP-14_W7.62mm_Socket_LongPads; moved to B.Cu
- J901, J902, J903, J904, J905, J906: footprint ao_tht:Jack_6.35mm_PJ_629HAN_slots -> AO_tht:Jack_6.35mm_PJ_629HAN_slots
- LED1: footprint ao_tht:LED_D5.0mm -> AO_tht:LED_D5.0mm
- R1, R10, R101, R102, R103, R104, R105, R106, R107, R108, R109, R11, R110, R12, R13, R16, R18, R19, R2, R20, R21, R22, R23, R24, R25, R26, R3, R6, R7, R8, R9, R901, R902: footprint ao_tht:R_Axial_DIN0207_L6.3mm_D2.5mm_P10.16mm_Horizontal -> AO_tht:R_Axial_DIN0207_L6.3mm_D2.5mm_P10.16mm_Horizontal; moved to B.Cu
- RV901, RV902, RV903, RV904: footprint ao_tht:Potentiometer_Alpha_16mm_Single_Vertical -> AO_tht:Potentiometer_Alpha_16mm_Single_Vertical
- SV101: footprint ao_tht:Power_Header -> AO_tht:Power_Header
- SW901: footprint ao_tht:SPDT-toggle-switch-1M-series -> AO_tht:SPDT-toggle-switch-1M-series
- TP901, TP902, TP903, TP904, TP905, TP906: footprint ao_tht:TestPoint_THTPad_D1.5mm_Drill0.7mm -> AO_tht:TestPoint_THTPad_D1.5mm_Drill0.7mm
- U1, U2, U7: footprint ao_tht:DIP-8_W7.62mm_Socket_LongPads -> AO_tht:DIP-8_W7.62mm_Socket_LongPads; moved to B.Cu
- U901: footprint ao_tht:TO-92_Inline_Wide -> AO_tht:TO-92_Inline_Wide; moved to B.Cu
- V101: footprint ao_tht:Vactrol_VTL5C -> AO_tht:Vactrol_VTL5C; moved to B.Cu
- VR1: footprint ao_tht:Potentiometer_Bourns_3362P_Vertical_screw_centered -> AO_tht:Potentiometer_Bourns_3362P_Vertical_screw_centered
- moved LED1 147.1 mm to (88.8, 73.5), turned to 180 degrees
- moved RV904 86.2 mm to (125.0, 40.0)
- moved R1 84.5 mm to (124.1, 134.3)
- moved R2 84.1 mm to (124.1, 129.2), turned to 0 degrees
- moved R26 77.5 mm to (92.4, 124.1), turned to 90 degrees
- moved Z$102 75.5 mm to (242.5, 60.9), turned to 180 degrees
- moved R7 72.2 mm to (124.1, 124.1)
- moved J906 67.3 mm to (262.5, 150.0)
- moved C109 66.3 mm to (194.0, 106.3), turned to 90 degrees
- moved R107 65.8 mm to (199.1, 100.0), turned to -90 degrees
- moved V101 61.6 mm to (230.8, 115.1)
- moved C903 60.6 mm to (118.8, 133.0), turned to 180 degrees
- moved C904 58.0 mm to (113.7, 117.8), turned to 180 degrees
- moved U1 57.4 mm to (111.2, 129.2), turned to 0 degrees
- moved R25 55.9 mm to (87.3, 114.0), turned to -90 degrees
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Connections:
- net Net-(C108-Pad1) renamed /Back board/TO_TANK_S_B
- net Net-(C110-Pad2) renamed /Back board/MIXPOT_WET_B
- net Net-(IC103-Pad8) renamed /Back board/MIXPOT_DRY_B
- net Net-(U901-Pad1) renamed +5V
- LED1 pad 1: Net-(LED1-Pad1) -> /Front board/VAC_AN_F
- LED1 pad 2: /Back board/VAC_AN_B -> Net-(LED1-A)
- U2 pad 1: /Front board/VAC_AN_F -> Net-(LED1-A)
- V101 pad 2: Net-(LED1-Pad1) -> /Back board/VAC_AN_B
Routing:
- net /Back board/CV_IN: track 25.3 -> 162.9 mm, vias 1 -> 0
- net /Back board/AUDIO_IN_1: track 29.6 -> 128.4 mm
- net Net-(LED1-Pad1): track 97.4 -> 0.00 mm, vias 1 -> 0
- net /Back board/VAC_CA_B: track 101.5 -> 20.7 mm
- net /Front board/TRIM_F: track 99.0 -> 26.5 mm
- net /Back board/TO_TANK: track 58.7 -> 128.0 mm, vias 1 -> 0
- net /Back board/TO_TANK_S_B: track 58.8 -> 126.3 mm
- net /Front board/AUDIO_IN_2: track 52.7 -> 120.0 mm, vias 1 -> 0
- net /Back board/AUDIO_IN_2: track 55.3 -> 116.0 mm
- net Net-(IC102B--): track 88.0 -> 27.5 mm
- net /Front board/AUDIO_IN_1: track 110.1 -> 50.1 mm
- net /Back board/EQ_POT_1_B: track 92.7 -> 41.1 mm, vias 1 -> 0
- net /Back board/MIXPOT_DRY_B: track 30.1 -> 74.4 mm, vias 0 -> 1
- net /Front board/FB_ON: track 56.6 -> 13.3 mm
- net /Front board/MIX: track 68.8 -> 29.4 mm
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Other:
- board size 165 x 159.5 mm -> 215 x 159.5 mm
- board text added: "Back board"
- board text added: "Circuit design by Tom Whitwell https://github.com/TomWhitwell/Spring-Reverb-Mk-2 CC-BY-SA"
- board text added: "Fill jumper if brick is not used"
- board text added: "Kosmo layout by Rich Holmes Feb 2022"
- board text added: "SPRING REVERB"
- board text added: "Spring Reverb Front board"
