File: Hardware/springReverbRev2/back.kicad_sch (KiCad schematic)
At the start: 54 parts, among them IC102 TL074, IC103 TL074, J901 AudioJack2_SwitchT, J902 AudioJack2, J903 AudioJack2, J904 AudioJack2, J905 AudioJack2_SwitchT, J906 AudioJack2, J917 DIP-8, J919 DIP-14, J920 DIP-14, U7 NE5532, U901 L78L05_TO92, X101 RCA, X102 RCA

Commit message: PCB revisions, Docs
Parts:
- added B902: Board, AO_tht:Board_Marker, symbol AO_symbols:Board
- C1, C101, C109, C2: footprint AO_tht:C_Disc_D3.0mm_W1.6mm_P2.50mm -> AO_tht:C_Radial_D8.0mm_H11.5mm_P3.50mm
- C108, C110, C3, C4: footprint AO_tht:C_Disc_D3.0mm_W1.6mm_P2.50mm -> AO_tht:C_Rect_L7.2mm_W2.5mm_P5.00mm_FKS2_FKP2_MKS2_MKP2
- J919, J920: SKU (none) -> A-004; Vendor (none) -> Tayda
Changed lines of the file:
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@@
   (title_block
     (title "Spring Reverb Rev 2")
+    (date "2023-03-17")
     (company "Music Thing Modular")
     (comment 1 "Kosmo version by Rich Holmes")
@@
   (junction (at 162.56 130.81) (diameter 0) (color 0 0 0 0)
   )
-  (junction (at 68.58 97.79) (diameter 0) (color 0 0 0 0)
-  )
   (junction (at 73.66 125.73) (diameter 0) (color 0 0 0 0)
   )
@@
     (stroke (width 0) (type default))
   )
-  (wire (pts (xy 67.31 97.79) (xy 68.58 97.79))
-    (stroke (width 0) (type default))
-  )
   (wire (pts (xy 218.44 41.91) (xy 208.28 41.91))
     (stroke (width 0) (type default))
@@
     (stroke (width 0) (type default))
   )
-  (wire (pts (xy 68.58 97.79) (xy 71.12 97.79))
+  (wire (pts (xy 67.31 97.79) (xy 71.12 97.79))
     (stroke (width 0) (type default))
   )
@@
       (effects (font (size 1.27 1.27)))
     )
-    (property "Footprint" "AO_tht:C_Disc_D3.0mm_W1.6mm_P2.50mm" (at 226.06 40.9448 0)
+    (property "Footprint" "AO_tht:C_Rect_L7.2mm_W2.5mm_P5.00mm_FKS2_FKP2_MKS2_MKP2" (at 226.06 40.9448 0)
       (effects (font (size 1.27 1.27)) hide)
     )
@@
   )
   (symbol (lib_id "AO_symbols:DIP-14") (at 97.79 190.5 0) (unit 1)
-    (in_bom yes) (on_board yes) (dnp no) (fields_autoplaced)
+    (in_bom yes) (on_board no) (dnp no) (fields_autoplaced)
     (property "Reference" "J919" (at 97.79 189.484 0)
       (effects (font (size 1.27 1.27)) hide)
@@
       (effects (font (size 1.27 1.27)) hide)
     )
+    (property "Vendor" "Tayda" (at 97.79 190.5 0)
+      (effects (font (size 1.27 1.27)) hide)
+    )
+    (property "SKU" "A-004" (at 97.79 190.5 0)
+      (effects (font (size 1.27 1.27)) hide)
+    )
     (instances
       (project "springReverbRev2"
@@
       (effects (font (size 1.778 1.5113)) (justify left bottom))
     )
-    (property "Footprint" "AO_tht:C_Disc_D3.0mm_W1.6mm_P2.50mm" (at 207.01 158.4452 0)
+    (property "Footprint" "AO_tht:C_Radial_D8.0mm_H11.5mm_P3.50mm" (at 207.01 158.4452 0)
       (effects (font (size 1.27 1.27)) hide)
     )
@@
       (effects (font (size 1.778 1.5113)) (justify left bottom))
     )
-    (property "Footprint" "AO_tht:C_Disc_D3.0mm_W1.6mm_P2.50mm" (at 207.01 138.1252 0)
+    (property "Footprint" "AO_tht:C_Radial_D8.0mm_H11.5mm_P3.50mm" (at 207.01 138.1252 0)
       (effects (font (size 1.27 1.27)) hide)
     )
@@
       (effects (font (size 1.27 1.27)))
     )
-    (property "Footprint" "AO_tht:C_Disc_D3.0mm_W1.6mm_P2.50mm" (at 160.02 148.8948 0)
+    (property "Footprint" "AO_tht:C_Rect_L7.2mm_W2.5mm_P5.00mm_FKS2_FKP2_MKS2_MKP2" (at 160.02 148.8948 0)
       (effects (font (size 1.27 1.27)) hide)
     )
@@
       (effects (font (size 1.27 1.27)))
     )
-    (property "Footprint" "AO_tht:C_Disc_D3.0mm_W1.6mm_P2.50mm" (at 210.82 53.6448 0)
+    (property "Footprint" "AO_tht:C_Rect_L7.2mm_W2.5mm_P5.00mm_FKS2_FKP2_MKS2_MKP2" (at 210.82 53.6448 0)
       (effects (font (size 1.27 1.27)) hide)
     )
@@
   )
   (symbol (lib_id "AO_symbols:DIP-8") (at 92.71 189.23 0) (unit 1)
-    (in_bom yes) (on_board yes) (dnp no) (fields_autoplaced)
+    (in_bom yes) (on_board no) (dnp no) (fields_autoplaced)
     (property "Reference" "J917" (at 92.71 187.96 0)
       (effects (font (size 1.27 1.27)) hide)
@@
       (effects (font (size 1.27 1.27)) (justify left))
     )
-    (property "Footprint" "AO_tht:C_Disc_D3.0mm_W1.6mm_P2.50mm" (at 74.6252 134.62 0)
+    (property "Footprint" "AO_tht:C_Rect_L7.2mm_W2.5mm_P5.00mm_FKS2_FKP2_MKS2_MKP2" (at 74.6252 134.62 0)
       (effects (font (size 1.27 1.27)) hide)
     )
@@
     )
   )
+  (symbol (lib_id "AO_symbols:Board") (at 130.81 199.39 0) (unit 1)
+    (in_bom no) (on_board yes) (dnp no) (fields_autoplaced)
+    (property "Reference" "B902" (at 137.16 198.755 0)
+      (effects (font (size 1.27 1.27)) (justify left))
+    )
+    (property "Value" "Board" (at 137.16 201.295 0)
+      (effects (font (size 1.27 1.27)) (justify left))
+    )
+    (property "Footprint" "AO_tht:Board_Marker" (at 130.81 199.39 0)
+      (effects (font (size 1.27 1.27)) hide)
+    )
+    (property "Datasheet" "" (at 130.81 199.39 0)
+      (effects (font (size 1.27 1.27)) hide)
+    )
+    (instances
+      (project "springReverbRev2"
+        (path "/7cc2117a-75f3-473b-aa3c-f6f0c8514e37/cb7e7ca4-1a75-4992-9aba-d7df48630a9d"
+          (reference "B902") (unit 1)
+        )
+      )
+    )
+  )
   (symbol (lib_id "AO_symbols:C") (at 38.1 157.48 0) (unit 1)
     (in_bom yes) (on_board yes) (dnp no) (fields_autoplaced)
@@
       (effects (font (size 1.27 1.27)) (justify left))
     )
-    (property "Footprint" "AO_tht:C_Disc_D3.0mm_W1.6mm_P2.50mm" (at 39.0652 161.29 0)
+    (property "Footprint" "AO_tht:C_Radial_D8.0mm_H11.5mm_P3.50mm" (at 39.0652 161.29 0)
       (effects (font (size 1.27 1.27)) hide)
     )
@@
   )
   (symbol (lib_id "AO_symbols:DIP-14") (at 102.87 190.5 0) (unit 1)
-    (in_bom yes) (on_board yes) (dnp no) (fields_autoplaced)
+    (in_bom yes) (on_board no) (dnp no) (fields_autoplaced)
     (property "Reference" "J920" (at 102.87 189.484 0)
       (effects (font (size 1.27 1.27)) hide)
@@
       (effects (font (size 1.27 1.27)) hide)
     )
+    (property "Vendor" "Tayda" (at 102.87 190.5 0)
+      (effects (font (size 1.27 1.27)) hide)
+    )
+    (property "SKU" "A-004" (at 102.87 190.5 0)
+      (effects (font (size 1.27 1.27)) hide)
+    )
     (instances
       (project "springReverbRev2"
@@
       (effects (font (size 1.27 1.27)) (justify right))
     )
-    (property "Footprint" "AO_tht:C_Disc_D3.0mm_W1.6mm_P2.50mm" (at 145.7452 151.13 0)
+    (property "Footprint" "AO_tht:C_Radial_D8.0mm_H11.5mm_P3.50mm" (at 145.7452 151.13 0)
       (effects (font (size 1.27 1.27)) hide)
     )
@@
         )
       )
-    )
-  )
-  (symbol (lib_id "power:PWR_FLAG") (at 68.58 97.79 180) (unit 1)
-    (in_bom yes) (on_board yes) (dnp no) (fields_autoplaced)
-    (property "Reference" "#FLG0905" (at 68.58 99.695 0)
-      (effects (font (size 1.27 1.27)) hide)
-    )
-    (property "Value" "PWR_FLAG" (at 68.58 102.2334 0)
-      (effects (font (size 1.27 1.27)))
-    )
-    (property "Footprint" "" (at 68.58 97.79 0)
-      (effects (font (size 1.27 1.27)) hide)
-    )
-    (property "Datasheet" "~" (at 68.58 97.79 0)
-      (effects (font (size 1.27 1.27)) hide)
-    )
-    (pin "1")
-    (instances
-      (project "springReverbRev2"
-        (path "/7cc2117a-75f3-473b-aa3c-f6f0c8514e37/cb7e7ca4-1a75-4992-9aba-d7df48630a9d"
-          (reference "#FLG0905") (unit 1)
-        )
-      )
