File: Hardware/springReverbRev2/front.kicad_sch (KiCad schematic)
At the start: 50 parts, among them J915 DIP-8, J916 DIP-8, SW901 SW_SPDT_MSM, U1 TL072, U2 TL072

Commit message: PCB revisions, Docs
Parts:
- added B901: Board, AO_tht:Board_Marker, symbol AO_symbols:Board
Changed lines of the file:
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@@
   )
   (symbol (lib_id "AO_symbols:DIP-8") (at 184.15 151.13 0) (unit 1)
-    (in_bom yes) (on_board yes) (dnp no) (fields_autoplaced)
+    (in_bom yes) (on_board no) (dnp no) (fields_autoplaced)
     (property "Reference" "J916" (at 184.15 149.86 0)
       (effects (font (size 1.27 1.27)) hide)
@@
   )
   (symbol (lib_id "AO_symbols:DIP-8") (at 179.07 151.13 0) (unit 1)
-    (in_bom yes) (on_board yes) (dnp no) (fields_autoplaced)
+    (in_bom yes) (on_board no) (dnp no) (fields_autoplaced)
     (property "Reference" "J915" (at 179.07 149.86 0)
       (effects (font (size 1.27 1.27)) hide)
@@
         )
       )
+    )
+  )
+  (symbol (lib_id "AO_symbols:Board") (at 116.84 184.15 0) (unit 1)
+    (in_bom no) (on_board yes) (dnp no) (fields_autoplaced)
+    (property "Reference" "B901" (at 123.19 183.515 0)
+      (effects (font (size 1.27 1.27)) (justify left))
+    )
+    (property "Value" "Board" (at 123.19 186.055 0)
+      (effects (font (size 1.27 1.27)) (justify left))
+    )
+    (property "Footprint" "AO_tht:Board_Marker" (at 116.84 184.15 0)
+      (effects (font (size 1.27 1.27)) hide)
+    )
+    (property "Datasheet" "" (at 116.84 184.15 0)
+      (effects (font (size 1.27 1.27)) hide)
+    )
+    (instances
+      (project "springReverbRev2"
+        (path "/7cc2117a-75f3-473b-aa3c-f6f0c8514e37/cb7e7ca4-1a75-4992-9aba-d7df48630a9d"
+          (reference "B901") (unit 1)
+        )
+        (path "/7cc2117a-75f3-473b-aa3c-f6f0c8514e37/757cdb0d-1f9d-4951-b906-b680c7b834f3"
+          (reference "B901") (unit 1)
+        )
+      )
