File: Hardware/springReverbRev2/panelmount.kicad_sch (KiCad schematic)
At the start: 2 parts, among them X103 RCA, X104 RCA

Commit message: PCB revisions, Docs
Parts:
- X103, X104: footprint AO_tht:Jack_6.35mm_PJ_629HAN_slots -> (none)
Other:
- company: (none) -> Music Thing Modular
- title: (none) -> Spring Reverb Rev 2
Changed lines of the file:
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@@
 (kicad_sch (version 20230121) (generator eeschema)
-  (paper "A4")
+  (paper "USLetter")
+  (title_block
+    (title "Spring Reverb Rev 2")
+    (company "Music Thing Modular")
+    (comment 1 "Kosmo version by Rich Holmes")
+  )
+  (junction (at 152.4 58.42) (diameter 0) (color 0 0 0 0)
+  )
+  (wire (pts (xy 152.4 58.42) (xy 156.21 58.42))
+    (stroke (width 0) (type default))
+  )
   (wire (pts (xy 151.13 55.88) (xy 152.4 55.88))
     (stroke (width 0) (type default))
@@
       (effects (font (size 1.27 1.27)) (justify right))
     )
-    (property "Footprint" "AO_tht:Jack_6.35mm_PJ_629HAN_slots" (at 124.46 57.15 0)
+    (property "Footprint" "" (at 124.46 57.15 0)
       (effects (font (size 1.27 1.27)) hide)
     )
@@
     )
   )
+  (symbol (lib_id "power:PWR_FLAG") (at 156.21 58.42 180) (unit 1)
+    (in_bom yes) (on_board yes) (dnp no) (fields_autoplaced)
+    (property "Reference" "#FLG0905" (at 156.21 60.325 0)
+      (effects (font (size 1.27 1.27)) hide)
+    )
+    (property "Value" "PWR_FLAG" (at 156.21 62.8634 0)
+      (effects (font (size 1.27 1.27)))
+    )
+    (property "Footprint" "" (at 156.21 58.42 0)
+      (effects (font (size 1.27 1.27)) hide)
+    )
+    (property "Datasheet" "~" (at 156.21 58.42 0)
+      (effects (font (size 1.27 1.27)) hide)
+    )
+    (pin "1")
+    (instances
+      (project "springReverbRev2"
+        (path "/7cc2117a-75f3-473b-aa3c-f6f0c8514e37/cb7e7ca4-1a75-4992-9aba-d7df48630a9d"
+          (reference "#FLG0905") (unit 1)
+        )
+        (path "/7cc2117a-75f3-473b-aa3c-f6f0c8514e37/d6ac4d33-ccdb-4ff9-b480-fe4304c892c2"
+          (reference "#FLG0905") (unit 1)
+        )
+      )
+    )
+  )
   (symbol (lib_id "AO_symbols:AudioJack2") (at 146.05 55.88 0) (mirror x) (unit 1)
     (in_bom yes) (on_board no) (dnp no)
@@
       (effects (font (size 1.27 1.27)) (justify right))
     )
-    (property "Footprint" "AO_tht:Jack_6.35mm_PJ_629HAN_slots" (at 146.05 55.88 0)
+    (property "Footprint" "" (at 146.05 55.88 0)
       (effects (font (size 1.27 1.27)) hide)
     )
